Commit message: Align scoop and support tool tips with TCP

File: assets/g1_scoop_endsupport/g1_29dof_rev_1_0_scoop_endsupport.urdf (robot description, URDF)
Before this commit: robot g1_29dof_rev_1_0_scoop_endsupport, 41 links, 40 joints
Links:
- link left_end_support_link: mass 0.462258829 -> 0.530869935; geometry collision box size=0.03 0.044 0.044; collision box size=0.2363 0.09 0.004
Joints:
- joint left_end_support_tcp_joint: origin xyz=0.180305 0 -0.0380589785 rpy=0 0 0 -> xyz=0.2483 0 -0.0141299543 rpy=0 0 0
- joint right_scoop_tcp_joint: origin xyz=0.180305 0 -0.0380589785 rpy=0 0 0 -> xyz=0.2483 0 -0.0141299543 rpy=0 0 0
