Commit message: Mount gripper tools facing inward and add a symmetric attention pose
- Rotate the scoop and end-support mounts +/-90 deg about the forward axis so their
  top faces point at the torso; mirror the rotation for the left/right swapped editor
  model and compute TCPs in the rotated tool links.
- Track the new model fingerprint as compatible with saved projects.
- Add Robot.attention: the default stand's base, legs and waist with the arms hanging
  at the sides (elbow 1.3 rad, shoulder roll +/-0.2 rad), so pinned feet stay put.
- Ship the tool meshes, preview/validation scripts and the added yaw preset group.

Co-Authored-By: Claude Sonnet 5.5 <noreply@anthropic.com>

File: assets/g1_scoop_endsupport/g1_29dof_rev_1_0_scoop_endsupport.urdf (robot description, URDF)
Before this commit: robot g1_29dof_rev_1_0_scoop_endsupport, 41 links, 40 joints
Joints:
- joint left_end_support_joint: origin xyz=0.0415 0 0 rpy=0 0 0 -> xyz=0.0415 0 0 rpy=1.57079633 0 0
- joint right_scoop_joint: origin xyz=0.0415 0 0 rpy=0 0 0 -> xyz=0.0415 0 0 rpy=-1.57079633 0 0

Commit message: Put the measured color lens position into the URDF d435_joint (moved 2, -5, -15 mm along the link axes) and reduce the PiP point cloud adjustment default to zero
Co-Authored-By: Claude Sonnet 5.5 <noreply@anthropic.com>

File: assets/g1_scoop_endsupport/g1_29dof_rev_1_0_scoop_endsupport.urdf (robot description, URDF)
Before this commit: robot g1_29dof_rev_1_0_scoop_endsupport, 41 links, 40 joints
Joints:
- joint d435_joint: origin xyz=0.0576235 0.01753 0.42987 rpy=0 0.8307767239493009 0 -> xyz=0.04789527 0.01253 0.4182786 rpy=0 0.8307767239493009 0

Commit message: Restore the original d435_joint and make the compare-view adjustment (2, -5, -16 mm) the point cloud origin default; fix the installer's stale-process match
Co-Authored-By: Claude Sonnet 5.5 <noreply@anthropic.com>

File: assets/g1_scoop_endsupport/g1_29dof_rev_1_0_scoop_endsupport.urdf (robot description, URDF)
Before this commit: robot g1_29dof_rev_1_0_scoop_endsupport, 41 links, 40 joints
Joints:
- joint d435_joint: origin xyz=0.04789527 0.01253 0.4182786 rpy=0 0.8307767239493009 0 -> xyz=0.0576235 0.01753 0.42987 rpy=0 0.8307767239493009 0
